File: MainPCB-HOTSWAP/EnvKB65HS.kicad_sch (KiCad schematic)
At the start: 157 parts

Commit message: updated pcb designs from upstream
Parts:
- added J1: Conn_01x04, Connector_PinSocket_2.54mm:PinSocket_1x04_P2.54mm_Vertical, symbol Connector_Generic:Conn_01x04
- added ST7: STABILIZER, Mounting_Keyboard_Stabilizer:Stabilizer_Cherry_MX_2u, symbol Mechanical:MountingHole
- D_0, D_1, D_10, D_11, D_12, D_13, D_14, D_15, D_16, D_17, D_18, D_19, D_2, D_20, D_21, D_22, D_23, D_24, D_25, D_26, D_27, D_28, D_29, D_3, D_30, D_31, D_32, D_33, D_34, D_35, D_36, D_37, D_38, D_39, D_4, D_40, D_41, D_42, D_43, D_44, D_45, D_46, D_47, D_48, D_49, D_5, D_50, D_51, D_52, D_53, D_54, D_55, D_56, D_57, D_58, D_59, D_6, D_60, D_61, D_62, D_63, D_64, D_65, D_66, D_67, D_68, D_69, D_7, D_70, D_8, D_9: value (none) -> 1n4148; footprint (none) -> Diode_SMD:D_SOD-123
- H0, H1, H2, H3, H4, H5: value (none) -> C2928180; footprint (none) -> MountingHole:MountingHole_3.5mm
- K_0, K_1, K_10, K_11, K_12, K_13, K_14, K_15, K_16, K_17, K_18, K_19, K_2, K_20, K_21, K_22, K_23, K_24, K_25, K_26, K_27, K_28, K_29, K_3, K_30, K_31, K_32, K_33, K_34, K_35, K_36, K_37, K_38, K_39, K_4, K_40, K_41, K_42, K_43, K_44, K_45, K_46, K_47, K_48, K_49, K_5, K_50, K_51, K_52, K_53, K_54, K_55, K_56, K_57, K_58, K_59, K_6, K_60, K_61, K_62, K_63, K_64, K_65, K_66, K_67, K_68, K_69, K_7, K_70, K_71, K_72, K_8, K_9: value (none) -> KEYSW; footprint (none) -> MX_Only:MXOnly-1U-Hotswap-Modified
- ST1, ST2, ST3, ST4, ST5, ST6: value (none) -> STABILIZER; footprint (none) -> Mounting_Keyboard_Stabilizer:Stabilizer_Cherry_MX_2u
- U0: value (none) -> Pico; footprint (none) -> MCU_RaspberryPi_and_Boards:RPi_Pico_SMD_TH
Connections:
- net GND: now also J1.1 (Pin_1); no longer H0.1, H1.1, H2.1, H3.1, H4.1, H5.1
- net USBVBUS: now reaches U0.40 (VBUS)
- net USBVBUS: now also J1.2 (Pin_2)
- net GPIO26 renamed I2C-SDA
- net I2C-SDA: now also J1.4 (Pin_4)
- net GPIO27 renamed I2C-SCL
- net I2C-SCL: now also J1.3 (Pin_3)
- no-connect marks 0 -> 6

Commit message: updated gerbers
Parts:
- H0, H1, H2, H3, H4, H5: footprint MountingHole:MountingHole_3.5mm -> MountingHole:MountingHole_3.2mm_M3
Changed lines of the file:
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@@
       (effects (font (size 1.27 1.27)) (justify left) hide)
     )
-    (property "Footprint" "MountingHole:MountingHole_3.5mm" (id 2) (at 542.29 71.12 0)
+    (property "Footprint" "MountingHole:MountingHole_3.2mm_M3" (id 2) (at 542.29 71.12 0)
       (effects (font (size 1.27 1.27)) hide)
     )
@@
       (effects (font (size 1.27 1.27)) (justify left) hide)
     )
-    (property "Footprint" "MountingHole:MountingHole_3.5mm" (id 2) (at 549.91 71.12 0)
+    (property "Footprint" "MountingHole:MountingHole_3.2mm_M3" (id 2) (at 549.91 71.12 0)
       (effects (font (size 1.27 1.27)) hide)
     )
@@
       (effects (font (size 1.27 1.27)) (justify left) hide)
     )
-    (property "Footprint" "MountingHole:MountingHole_3.5mm" (id 2) (at 557.53 71.12 0)
+    (property "Footprint" "MountingHole:MountingHole_3.2mm_M3" (id 2) (at 557.53 71.12 0)
       (effects (font (size 1.27 1.27)) hide)
     )
@@
       (effects (font (size 1.27 1.27)) (justify left) hide)
     )
-    (property "Footprint" "MountingHole:MountingHole_3.5mm" (id 2) (at 565.15 71.12 0)
+    (property "Footprint" "MountingHole:MountingHole_3.2mm_M3" (id 2) (at 565.15 71.12 0)
       (effects (font (size 1.27 1.27)) hide)
     )
@@
       (effects (font (size 1.27 1.27)) (justify left) hide)
     )
-    (property "Footprint" "MountingHole:MountingHole_3.5mm" (id 2) (at 572.77 71.12 0)
+    (property "Footprint" "MountingHole:MountingHole_3.2mm_M3" (id 2) (at 572.77 71.12 0)
       (effects (font (size 1.27 1.27)) hide)
     )
@@
       (effects (font (size 1.27 1.27)) (justify left) hide)
     )
-    (property "Footprint" "MountingHole:MountingHole_3.5mm" (id 2) (at 580.39 71.12 0)
+    (property "Footprint" "MountingHole:MountingHole_3.2mm_M3" (id 2) (at 580.39 71.12 0)
       (effects (font (size 1.27 1.27)) hide)
     )
@@
     )
     (path "/00000000-0000-0000-0000-000060ac66fb"
-      (reference "H0") (unit 1) (value "C2928180") (footprint "MountingHole:MountingHole_3.5mm")
+      (reference "H0") (unit 1) (value "C2928180") (footprint "MountingHole:MountingHole_3.2mm_M3")
     )
     (path "/00000000-0000-0000-0000-000060acbe92"
-      (reference "H1") (unit 1) (value "C2928180") (footprint "MountingHole:MountingHole_3.5mm")
+      (reference "H1") (unit 1) (value "C2928180") (footprint "MountingHole:MountingHole_3.2mm_M3")
     )
     (path "/00000000-0000-0000-0000-000060ae412b"
-      (reference "H2") (unit 1) (value "C2928180") (footprint "MountingHole:MountingHole_3.5mm")
+      (reference "H2") (unit 1) (value "C2928180") (footprint "MountingHole:MountingHole_3.2mm_M3")
     )
     (path "/00000000-0000-0000-0000-000060afc1c3"
-      (reference "H3") (unit 1) (value "C2928180") (footprint "MountingHole:MountingHole_3.5mm")
+      (reference "H3") (unit 1) (value "C2928180") (footprint "MountingHole:MountingHole_3.2mm_M3")
     )
     (path "/00000000-0000-0000-0000-000060b142b5"
-      (reference "H4") (unit 1) (value "C2928180") (footprint "MountingHole:MountingHole_3.5mm")
+      (reference "H4") (unit 1) (value "C2928180") (footprint "MountingHole:MountingHole_3.2mm_M3")
     )
     (path "/00000000-0000-0000-0000-000060b2c4b8"
-      (reference "H5") (unit 1) (value "C2928180") (footprint "MountingHole:MountingHole_3.5mm")
+      (reference "H5") (unit 1) (value "C2928180") (footprint "MountingHole:MountingHole_3.2mm_M3")
     )
     (path "/71e681d9-af3d-408d-a1f2-12eb69afec3c"
