File: MainPCB/EnvKB65.kicad_pcb (KiCad board)
At the start: 2 copper layers, 320.8 x 99.3 mm, 157 parts, among them U0 Pico

Commit message: cleaned up repo and updated readme
Other:
- board text added: "http://github.com/Envious-Data/Env-KB65M https://github.com/Envious-Data/EnvKB-QMK"
- board text removed: "http://github.com/Envious-Data/Env-KB65M https://github.com/Envious-Data/EnvKB-QMK https://envious.design/firmwares/"
